Commit message: wheel addiction

File: description/robot_core.xacro (robot description, xacro)
@@ -13,6 +13,8 @@
         <color rgba="0 0 0 1"/>
     </material>
+<!-- БАЗА LINK -->
     <link name="base_link">
     </link>
+<!--  CHASSIS LINK  -->
     <joint name="chassis_joint" type="fixed">
         <parent link="base_link"/>
@@ -29,3 +31,33 @@
         </visual>
     </link>
+<!-- LEFT WHEEL LINK -->
+    <joint name="left_wheel_joint" type="continuous">
+        <parent link="base_link"/>
+        <child link="left_wheel"/>
+        <origin xyz="0 0.175 0" rpy="-${pi/2} 0 0"/>
+        <axis xyz="0 0 1"/>
+    </joint>
+    <link name="left_wheel">
+        <visual>
+            <geometry>
+                <cylinder radius="0.05" length="0.04"/>
+            </geometry>
+            <material name="blue"/>
+        </visual>
+    </link>
+<!-- RIGHT WHEEL LINK -->
+    <joint name="right_wheel_joint" type="continuous">
+        <parent link="base_link"/>
+        <child link="right_wheel"/>
+        <origin xyz="0 -0.175 0" rpy="${pi/2} 0 0"/>
+        <axis xyz="0 0 -1"/>
+    </joint>
+    <link name="right_wheel">
+        <visual>
+            <geometry>
+                <cylinder radius="0.05" length="0.04"/>
+            </geometry>
+            <material name="blue"/>
+        </visual>
+    </link>
 </robot>

Commit message: caster

File: description/robot_core.xacro (robot description, xacro)
@@ -61,3 +61,17 @@
         </visual>
     </link>
+<!-- CASTER WHEEL LINK -->
+    <joint name="caster_wheel_joint" type="fixed">
+        <parent link="chassis"/>
+        <child link="caster_wheel"/>
+        <origin xyz="0.24 0 0">
+    </joint>
+    <link name="caster_wheel">
+        <visual>
+            <geometry>
+                <sphere radius="0.85"/>
+            </geometry>
+            <material name="black"/>
+        </visual>
+    </link>
 </robot>

Commit message: claster fix line86

File: description/robot_core.xacro (robot description, xacro)
@@ -65,5 +65,5 @@
         <parent link="chassis"/>
         <child link="caster_wheel"/>
-        <origin xyz="0.24 0 0">
+        <origin xyz="0.24 0 0"/>
     </joint>
     <link name="caster_wheel">

Commit message: caster fix radius

File: description/robot_core.xacro (robot description, xacro)
@@ -70,5 +70,5 @@
         <visual>
             <geometry>
-                <sphere radius="0.85"/>
+                <sphere radius="0.05"/>
             </geometry>
             <material name="black"/>

Commit message: добавил коллизию не знаю че это

File: description/robot_core.xacro (robot description, xacro)
@@ -30,4 +30,10 @@
             <material name="white"/>
         </visual>
+        <collision>
+            <origin xyz="0.15 0 0.075"/>
+            <geometry>
+                <box size="0.3 0.3 0.15"/>
+            </geometry>
+        </collision>
     </link>
 <!-- LEFT WHEEL LINK -->
@@ -45,4 +51,9 @@
             <material name="blue"/>
         </visual>
+        <collision>
+            <geometry>
+                <cylinder radius="0.05" length="0.04"/>
+            </geometry>
+        </collision>
     </link>
 <!-- RIGHT WHEEL LINK -->
@@ -60,4 +71,9 @@
             <material name="blue"/>
         </visual>
+        <collision>
+            <geometry>
+                <cylinder radius="0.05" length="0.04"/>
+            </geometry>
+        </collision>
     </link>
 <!-- CASTER WHEEL LINK -->
@@ -74,4 +90,9 @@
             <material name="black"/>
         </visual>
+        <collision>
+            <geometry>
+                <sphere radius="0.05"/>
+            </geometry>
+        </collision>
     </link>
 </robot>

Commit message: инерция

File: description/robot_core.xacro (robot description, xacro)
@@ -1,4 +1,5 @@
 <?xml version="1.0"?>
 <robot xmlns:xacro="http://www.ros.org/wiki/xacro">
+    <xacro:include filename+"inertial_macros.xacro"/>
     <material name="white">
         <color rgba="1 1 1 1"/>
@@ -36,4 +37,7 @@
             </geometry>
         </collision>
+        <xacro:inertial_box mass="0.5" x="0.3" y="0.3" z="0.15">
+            <origin xyz="0.15 0 0.075" rpy="0 0 0"/>
+        </xacro:inertial_box>
     </link>
 <!-- LEFT WHEEL LINK -->
@@ -56,4 +60,7 @@
             </geometry>
         </collision>
+        <xacro:inertial_cylinder mass="0.1" length="0.04" radius="0.05">
+            <origin xyz="0 0 0" rpy="0 0 0"/>
+        </xacro:inertial_cylinder>
     </link>
 <!-- RIGHT WHEEL LINK -->
@@ -76,4 +83,7 @@
             </geometry>
         </collision>
+        <xacro:inertial_cylinder mass="0.1" length="0.04" radius="0.05">
+            <origin xyz="0 0 0" rpy="0 0 0"/>
+        </xacro:inertial_cylinder>
     </link>
 <!-- CASTER WHEEL LINK -->
@@ -95,4 +105,7 @@
             </geometry>
         </collision>
+        <xacro:inertial_sphere mass="0.1" radius="0.5">
+            <origin xyz="0 0 0" rpy="0 0 0"/>
+        </xacro:inertial_sphere>
     </link>
 </robot>

Commit message: pomenyal razmeri

File: description/robot_core.xacro (robot description, xacro)
@@ -25,7 +25,7 @@
     <link name="chassis">
         <visual>
-            <origin xyz="0.15 0 0.075"/>
+            <origin xyz="0 0 0.13"/>
             <geometry>
-                <box size="0.3 0.3 0.15"/>
+                <box size="0.4 0.4 0.26"/>
             </geometry>
             <material name="white"/>
@@ -37,6 +37,6 @@
             </geometry>
         </collision>
-        <xacro:inertial_box mass="0.5" x="0.3" y="0.3" z="0.15">
-            <origin xyz="0.15 0 0.075" rpy="0 0 0"/>
+        <xacro:inertial_box mass="0.5" x="0.4" y="0.4" z="0.26">
+            <origin xyz="0 0 0.13" rpy="0 0 0"/>
         </xacro:inertial_box>
     </link>
@@ -45,5 +45,5 @@
         <parent link="base_link"/>
         <child link="left_wheel"/>
-        <origin xyz="0 0.175 0" rpy="-${pi/2} 0 0"/>
+        <origin xyz="0 0.2 0" rpy="-${pi/2} 0 0"/>
         <axis xyz="0 0 1"/>
     </joint>
@@ -68,5 +68,5 @@
         <parent link="base_link"/>
         <child link="right_wheel"/>
-        <origin xyz="0 -0.175 0" rpy="${pi/2} 0 0"/>
+        <origin xyz="0 -0.2 0" rpy="${pi/2} 0 0"/>
         <axis xyz="0 0 -1"/>
     </joint>
@@ -91,5 +91,5 @@
         <parent link="chassis"/>
         <child link="caster_wheel"/>
-        <origin xyz="0.24 0 0"/>
+        <origin xyz="-0.1 0 0"/>
     </joint>
     <link name="caster_wheel">

Commit message: add colors

File: description/robot_core.xacro (robot description, xacro)
@@ -41,4 +41,7 @@
         </xacro:inertial_box>
     </link>
+    <gazebo reference="chassis">
+        <material>Gazebo/White</material>
+    </gazebo>
 <!-- LEFT WHEEL LINK -->
     <joint name="left_wheel_joint" type="continuous">
@@ -64,4 +67,7 @@
         </xacro:inertial_cylinder>
     </link>
+    <gazebo reference="left_wheel">
+        <material>Gazebo/Blue</material>
+    </gazebo>
 <!-- RIGHT WHEEL LINK -->
     <joint name="right_wheel_joint" type="continuous">
@@ -87,4 +93,7 @@
         </xacro:inertial_cylinder>
     </link>
+    <gazebo reference="right_wheel">
+        <material>Gazebo/Blue</material>
+    </gazebo>
 <!-- CASTER WHEEL LINK -->
     <joint name="caster_wheel_joint" type="fixed">
@@ -109,3 +118,6 @@
         </xacro:inertial_sphere>
     </link>
+    <gazebo reference="caster_wheel">
+        <material>Gazebo/Black</material>
+    </gazebo>
 </robot>

Commit message: fixing bot model

File: description/robot_core.xacro (robot description, xacro)
@@ -25,5 +25,5 @@
     <link name="chassis">
         <visual>
-            <origin xyz="0 0 0.13"/>
+            <origin xyz="0.2 0 0.13"/>
             <geometry>
                 <box size="0.4 0.4 0.26"/>
@@ -32,11 +32,11 @@
         </visual>
         <collision>
-            <origin xyz="0.15 0 0.075"/>
+            <origin xyz="0.2 0 0.13"/>
             <geometry>
-                <box size="0.3 0.3 0.15"/>
+                <box size="0.4 0.4 0.26"/>
             </geometry>
         </collision>
-        <xacro:inertial_box mass="0.5" x="0.4" y="0.4" z="0.26">
-            <origin xyz="0 0 0.13" rpy="0 0 0"/>
+        <xacro:inertial_box mass="0.8" x="0.4" y="0.4" z="0.26">
+            <origin xyz="0.2 0 0.13" rpy="0 0 0"/>
         </xacro:inertial_box>
     </link>
@@ -48,5 +48,5 @@
         <parent link="base_link"/>
         <child link="left_wheel"/>
-        <origin xyz="0 0.2 0" rpy="-${pi/2} 0 0"/>
+        <origin xyz="0 0.22 0" rpy="-${pi/2} 0 0"/>
         <axis xyz="0 0 1"/>
     </joint>
@@ -74,5 +74,5 @@
         <parent link="base_link"/>
         <child link="right_wheel"/>
-        <origin xyz="0 -0.2 0" rpy="${pi/2} 0 0"/>
+        <origin xyz="0 -0.22 0" rpy="${pi/2} 0 0"/>
         <axis xyz="0 0 -1"/>
     </joint>
@@ -100,5 +100,5 @@
         <parent link="chassis"/>
         <child link="caster_wheel"/>
-        <origin xyz="-0.1 0 0"/>
+        <origin xyz="0.3 0 0"/>
     </joint>
     <link name="caster_wheel">

Commit message: lidar sdelal

File: description/robot_core.xacro (robot description, xacro)
@@ -13,4 +13,7 @@
     <material name="black">
         <color rgba="0 0 0 1"/>
+    </material>
+    <material name="red">
+        <color rgba="1 0 0 1"/>
     </material>
 <!-- БАЗА LINK -->
